Commit message: the final version

File: robot_model/urdf/robot_model.urdf (robot description, URDF)
Before this commit: robot robot_model, 20 links, 19 joints
Links:
- link link_0_x: geometry visual mesh filename=package://robot_model/mesh/tisch-und-base1.obj scale=1 1 1

File: robot_model/urdf/simple_box.urdf (robot description, URDF)
Before this commit: robot simple_box, 1 links, 0 joints
Links:
- added link base_link; visual cylinder length=0.01 radius=0.2
- link my_box: mass 1.0 -> None; geometry collision mesh filename=package://robot_model/mesh/L0.obj scale=1 1 1; visual mesh filename=package://robot_model/mesh/L0.obj scale=1 1 1
Joints:
- added joint joint_0: type fixed, parent base_link, child my_box, origin xyz=0 0 0 rpy=0 0 0
